File: choc/pcb/swoop-choc.kicad_pcb (KiCad board)
At the start: 2 copper layers, 108.8 x 88 mm, 67 parts, among them J1 TRRS, SW1 Choc, SW10 Choc, SW11 Choc, SW12 Choc, SW13 Choc, SW14 Choc, SW15 Choc, SW16 Choc, SW17 Choc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

Commit message: Reorganised the Choc
Parts:
- BT1: footprint jmnw:Battery_pads_reversible_2 -> swoop:Battery_pads_reversible
- L1, L10, L11, L12, L13, L14, L15, L16, L17, L2, L3, L4, L5, L6, L7, L8, L9: footprint jmnw:sk6812_mini_e_rev -> swoop:SK6812_Mini_E
- PSW1: footprint jmnw:Power_reversible -> swoop:Power
- Ref** (x2): footprint jmnw:M2_hole_3.5mm_2mm -> swoop:M2_hole_3.5mm
- moved BT1 0.60 mm to (155.4, 118.2)
