File: choc/plates/base-plate/one-fell-swoop-base-plate.kicad_pcb (KiCad board)
At the start: 2 copper layers, 108.8 x 88 mm, 72 parts, among them J1 TRRS, SW1 Choc_base_cutout, SW10 Choc_base_cutout, SW11 Choc_base_cutout, SW12 Choc_base_cutout, SW13 Choc_base_cutout, SW14 Choc_base_cutout, SW15 Choc_base_cutout, SW16 Choc_base_cutout, SW17 Choc_base_cutout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

Commit message: Reorganised the Choc
Parts:
- B1, B2, B3, B4: renamed from H2; footprint jmnw:M2_hole_3.5mm_2mm -> swoop:Bumper_cutout
- D1, D10, D11, D12, D13, D14, D15, D16, D17, D2, D3, D4 (x2), D5, D6, D7, D8, D9 (x2), ED1: footprint jmnw:D3_SMD_cutout -> swoop:D3_SMD_cutout
- D18: renamed from D14; footprint jmnw:D3_SMD_cutout -> swoop:D3_SMD_cutout
- EN1: footprint jmnw:RotaryEncoder_cutout -> swoop:RotaryEncoder_cutout
- EN2: footprint jmnw:RollerEncoder_cutout -> swoop:RollerEncoder_cutout
- G***: footprint jmnw:ferris-rust -> swoop:Ferris_rust_logos
- H1, H2, H3, H4 (x2): footprint jmnw:M2_hole_3.5mm_2mm -> swoop:M2_hole_3.5mm
- J1: footprint jmnw:TRRS-3pin_cutout -> swoop:TRRS-3pin_cutout
- L1, L10, L11, L12, L13, L14, L15, L16, L17, L2, L3, L4, L5, L6, L7, L8, L9: footprint jmnw:SK6812_Mini_E_cutout -> swoop:SK6812_Mini_E_cutout
- O1: footprint jmnw:OLED_cutout -> swoop:OLED_cutout
- Ref** (x2): footprint jmnw:M2_hole_3.5mm_2mm_cutout -> swoop:M2_hole_3.5mm_cutout
- SW1, SW10, SW11, SW12, SW13, SW14, SW15, SW16, SW17, SW2, SW3, SW4, SW5, SW6, SW7, SW8, SW9: value Choc_base_cutout -> Choc_cutout; footprint jmnw:Choc_base_cutout -> swoop:Choc_cutout
- U1: footprint jmnw:ProMicro_cutout -> swoop:ProMicro_cutout
