File: choc/plates/cover/one-fell-swoop-cover.kicad_pcb (KiCad board)
At the start: 2 copper layers, 18.3 x 54.2 mm, 2 parts

Commit message: Reorganised the Choc
Parts:
- Ref** (x2): footprint jmnw:M2_hole_2.3mm -> swoop:M2_hole_3.5mm
Changed lines of the file:
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@@
   )
   (net 0 "")
-  (footprint "jmnw:M2_hole_2.3mm" (layer "F.Cu")
+  (footprint "swoop:M2_hole_3.5mm" (layer "F.Cu")
     (at 156.068168 79.871776)
     (descr "Mounting Hole 2.2mm, no annular, M2")
@@
       (effects (font (size 1 1) (thickness 0.15)))
     )
-    (pad "" np_thru_hole circle locked (at 0 0) (size 2.3 2.3) (drill 2.3) (layers *.Cu *.Mask))
+    (pad "" thru_hole circle (at 0 0) (size 3.5 3.5) (drill 2.2) (layers *.Cu *.Mask))
   )
-  (footprint "jmnw:M2_hole_2.3mm" (layer "F.Cu")
+  (footprint "swoop:M2_hole_3.5mm" (layer "F.Cu")
     (at 165.884619 129.04088)
     (descr "Mounting Hole 2.2mm, no annular, M2")
@@
       (effects (font (size 1 1) (thickness 0.15)))
     )
-    (pad "" np_thru_hole circle locked (at 0 0) (size 2.3 2.3) (drill 2.3) (layers *.Cu *.Mask))
+    (pad "" thru_hole circle (at 0 0) (size 3.5 3.5) (drill 2.2) (layers *.Cu *.Mask))
   )
   (gr_line (start 159.568275 81.871667) (end 170.849214 81.871494) (layer "Edge.Cuts") (width 0.05))
   (gr_line (start 171.849217 82.87149) (end 171.84911 119.412056) (layer "Edge.Cuts") (width 0.05))
   (gr_arc (start 156.06811 77.371599) (mid 157.835919 78.103881) (end 158.568099 79.871733) (layer "Edge.Cuts") (width 0.05))
-  (gr_arc (start 168.05025 130.290667) (mid 166.532164 131.455465) (end 164.635077 131.205654) (layer "Edge.Cuts") (width 0.05))
+  (gr_arc (start 168.05025 130.290667) (mid 166.532163 131.455465) (end 164.635077 131.205654) (layer "Edge.Cuts") (width 0.05))
   (gr_arc (start 153.567977 79.871588) (mid 154.300279 78.1038) (end 156.06811 77.371599) (layer "Edge.Cuts") (width 0.05))
   (gr_line (start 158.568099 79.871733) (end 158.568272 80.871671) (layer "Edge.Cuts") (width 0.05))
