File: choc/plates/switch-plate/one-fell-swoop-switch-plate.kicad_pcb (KiCad board)
At the start: 2 copper layers, 103.2 x 88 mm, 22 parts, among them SW1 Choc cutout, SW10 Choc cutout, SW11 Choc cutout, SW12 Choc cutout, SW13 Choc cutout, SW14 Choc cutout, SW15 Choc cutout, SW16 Choc cutout, SW17 Choc cutout, SW2 Choc cutout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

Commit message: Reorganised the Choc
Parts:
- H1, H2, H3, H4 (x2): footprint jmnw:M2_hole_3.5mm_2mm -> swoop:M2_hole_3.5mm
- SW1, SW10, SW11, SW12, SW13, SW14, SW15, SW16, SW17, SW2, SW3, SW4, SW5, SW6, SW7, SW8, SW9: footprint jmnw:Choc_cutout -> swoop:Choc_cutout
