File: pcbs/swoop/swoop.kicad_sch (KiCad schematic)
At the start: 60 parts, among them J1 TRRS, SW1 Choc, SW10 Choc, SW11 Choc, SW12 Choc, SW13 Choc, SW14 Choc, SW15 Choc, SW16 Choc, SW17 Choc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

Commit message: Fixed the cover
Other:
- title: One Fell Swoop -> Swoop
Changed lines of the file:
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@@
   (paper "A4")
   (title_block
-    (title "One Fell Swoop")
-    (date "2022-02-02")
-    (rev "0.4")
+    (title "Swoop")
+    (date "2022-02-03")
+    (rev "0.4.1")
     (company "jmnw")
   )
