File: pcbs/howarya/howarya.kicad_pcb (KiCad board)
At the start: 2 copper layers, 114 x 97.8 mm, 73 parts, among them J1 TRRS, SW1 MX, SW10 MX, SW11 MX, SW12 MX, SW13 MX, SW14 MX, SW15 MX, SW16 MX, SW17 MX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

Commit message: Name change
Other:
- board text added: "Howarya? v0.2.1 https://github.com/jimmerricks/swoop"
- board text removed: "Swoop MX v0.2 https://github.com/jimmerricks/swoop"
Changed lines of the file:
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@@
   (paper "A4")
   (title_block
-    (title "Swoop MX")
-    (date "2021-12-18")
-    (rev "0.2")
+    (title "Howarya?")
+    (date "2022-02-03")
+    (rev "0.2.1")
     (company "jmnw")
   )
@@
     (fp_line (start -4.2 6.4) (end -3 6.4) (layer "B.SilkS") (width 0.4))
     (fp_arc (start 3.016318 1.55) (mid 2.130713 2.910207) (end 0.6 3.45) (layer "B.SilkS") (width 1))
-    (fp_arc (start 5.65 4.699999) (mid 4.993504 6.084925) (end 3.550001 6.6) (layer "B.SilkS") (width 0.15))
+    (fp_arc (start 5.65 4.699999) (mid 4.993504 6.084924) (end 3.550001 6.6) (layer "B.SilkS") (width 0.15))
     (fp_arc (start 2.616318 1.121471) (mid 1.868709 2.486118) (end 0.4 3) (layer "B.SilkS") (width 0.15))
     (fp_line (start 4.35 6.6) (end -3.800001 6.6) (layer "F.SilkS") (width 0.15))
@@
   (gr_line (start 161.817872 157.127673) (end 174.540128 135.091885) (layer "Edge.Cuts") (width 0.05))
   (gr_arc (start 172.287011 87.98281) (mid 172.872853 86.568559) (end 174.287148 85.982823) (layer "Edge.Cuts") (width 0.05))
-  (gr_text "Swoop MX v0.2\nhttps://github.com/jimmerricks/swoop" (at 168.090207 95.278026 90) (layer "B.SilkS")
+  (gr_text "Howarya? v0.2.1\nhttps://github.com/jimmerricks/swoop" (at 168.090207 95.278026 90) (layer "B.SilkS")
     (effects (font (size 0.8 0.8) (thickness 0.1)) (justify left mirror))
   )
-  (gr_text "Swoop MX v0.2\nhttps://github.com/jimmerricks/swoop" (at 168.090203 119.338026 90) (layer "F.SilkS")
+  (gr_text "Howarya? v0.2.1\nhttps://github.com/jimmerricks/swoop" (at 168.090203 119.338026 90) (layer "F.SilkS")
     (effects (font (size 0.8 0.8) (thickness 0.1)) (justify left))
   )

Commit message: Removed LED strip and normalised LED order.
Parts:
- removed JP1: PKRGB bypass, swoop:Jumper
- removed JP2: LED bypass, swoop:Jumper
- removed LS1: LED Strip, swoop:StripLED
Connections:
- L10 pad 2: Net-(L10-Pad2) -> Net-(L5-Pad4)
- L13 pad 2: Net-(L12-Pad4) -> Net-(L8-Pad4)
- L13 pad 4: Net-(L13-Pad4) -> Net-(L17-Pad2)
- L14 pad 2: Net-(L13-Pad4) -> Net-(L17-Pad4)
- L14 pad 4: l14i -> Net-(L14-Pad4)
- L15 pad 2: strip -> Net-(L10-Pad4)
- L15 pad 4: Net-(L10-Pad2) -> Net-(L18-Pad2)
- L16 pad 2: l14i -> unconnected-(L16-Pad2)
- L16 pad 4: l17o -> Net-(L1-Pad2)
- L17 pad 2: l17o -> Net-(L17-Pad2)
- L18 pad 2: Net-(L17-Pad4) -> Net-(L18-Pad2)
- L3 pad 2: Net-(L3-Pad2) -> Net-(L2-Pad4)
- L3 pad 4: Net-(L2-Pad2) -> Net-(L3-Pad4)
- L5 pad 2: Net-(L10-Pad4) -> Net-(L4-Pad4)
- L5 pad 4: Net-(L4-Pad2) -> Net-(L5-Pad4)
- L7 pad 2: Net-(L2-Pad4) -> Net-(L12-Pad4)
- L7 pad 4: Net-(L1-Pad2) -> Net-(L2-Pad2)
- L8 pad 2: Net-(L8-Pad2) -> Net-(L3-Pad4)
- L8 pad 4: Net-(L3-Pad2) -> Net-(L8-Pad4)
- L9 pad 2: Net-(L4-Pad4) -> Net-(L14-Pad4)
- L9 pad 4: Net-(L8-Pad2) -> Net-(L4-Pad2)
Routing:
- net Net-(L1-Pad2): track 39.5 -> 118.5 mm
- net Net-(L17-Pad2): track 0.00 -> 65.2 mm, vias 0 -> 2
- net l14i: track 54.9 -> 0.00 mm, vias 2 -> 0
- net Net-(L18-Pad2): track 0.00 -> 38.9 mm
- net Net-(L13-Pad4): track 38.5 -> 0.00 mm, vias 2 -> 0
- net l17o: track 37.8 -> 0.00 mm
- net strip: track 27.2 -> 0.00 mm
- net Net-(L14-Pad4): track 0.00 -> 25.8 mm
- net Net-(L10-Pad2): track 24.1 -> 0.00 mm
- net Net-(L3-Pad2): track 24.1 -> 0.00 mm
- net GND: track 521.4 -> 498.6 mm, vias 10 -> 9
- net Net-(L3-Pad4): track 0.00 -> 19.4 mm
- net Net-(L8-Pad4): track 0.00 -> 19.4 mm
- net Net-(L5-Pad4): track 0.00 -> 19.4 mm
- net VCC: track 495.7 -> 478.7 mm
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Other:
- board text added: "Howarya? v0.2.2 https://github.com/jimmerricks/swoop"
- board text removed: "Howarya? v0.2.1 https://github.com/jimmerricks/swoop"
