File: pcbs/plates/plates.kicad_pcb (KiCad board)
At the start: 2 copper layers, 108.1 x 88.5 mm, 8 parts

Commit message: small update to readme and plates
Parts:
- removed Ref** (x2): Val**, chocolad:M2_hole_3.5mm
- removed Ref**: Val**, swoop:M2_hole_3.5mm
Other:
- outline, holes or cut-outs redrawn
Changed lines of the file:
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@@
   (paper "A4")
   (title_block
-    (title "Swoop Choc")
-    (date "2023-05-28")
-    (rev "0.4.2")
-    (company "jmnw")
+    (title "Arkenswoop")
+    (date "2023-06-03")
+    (rev "0.4.3")
+    (company "lexplt")
   )
   (layers
@@
     (pad "" thru_hole circle (at 0 0) (size 4.2 4.2) (drill 3.8) (layers "*.Cu" "*.Mask"))
   )
-  (footprint "chocolad:M2_hole_3.5mm" (layer "F.Cu")
-    (at 169.385693 81.98964)
-    (descr "Mounting Hole 2.2mm, no annular, M2")
-    (tags "mounting hole 2.2mm no annular m2")
-    (attr exclude_from_pos_files exclude_from_bom)
-    (fp_text reference "Ref**" (at -0.95 -0.55) (layer "F.Fab") hide
-        (effects (font (size 1 1) (thickness 0.15)))
-    )
-    (fp_text value "Val**" (at 0 0.55) (layer "F.Fab") hide
-        (effects (font (size 1 1) (thickness 0.15)))
-    )
-    (fp_text user "${REFERENCE}" (at 0.3 0) (layer "F.Fab")
-        (effects (font (size 1 1) (thickness 0.15)))
-    )
-    (pad "" thru_hole circle (at 0 0) (size 3.5 3.5) (drill 2.2) (layers "*.Cu" "*.Mask"))
-  )
-  (footprint "chocolad:M2_hole_3.5mm" (layer "F.Cu")
-    (at 154.604371 81.990097)
-    (descr "Mounting Hole 2.2mm, no annular, M2")
-    (tags "mounting hole 2.2mm no annular m2")
-    (attr exclude_from_pos_files exclude_from_bom)
-    (fp_text reference "Ref**" (at -0.95 -0.55) (layer "F.Fab") hide
-        (effects (font (size 1 1) (thickness 0.15)))
-    )
-    (fp_text value "Val**" (at 0 0.55) (layer "F.Fab") hide
-        (effects (font (size 1 1) (thickness 0.15)))
-    )
-    (fp_text user "${REFERENCE}" (at 0.3 0) (layer "F.Fab")
-        (effects (font (size 1 1) (thickness 0.15)))
-    )
-    (pad "" thru_hole circle (at 0 0) (size 3.5 3.5) (drill 2.2) (layers "*.Cu" "*.Mask"))
-  )
-  (footprint "swoop:M2_hole_3.5mm" (layer "F.Cu")
-    (at 165.490722 131.887874)
-    (descr "Mounting Hole 2.2mm, no annular, M2")
-    (tags "mounting hole 2.2mm no annular m2")
-    (attr exclude_from_pos_files exclude_from_bom)
-    (fp_text reference "Ref**" (at -0.95 -0.55) (layer "F.Fab") hide
-        (effects (font (size 1 1) (thickness 0.15)))
-    )
-    (fp_text value "Val**" (at 0 0.55) (layer "F.Fab") hide
-        (effects (font (size 1 1) (thickness 0.15)))
-    )
-    (fp_text user "${REFERENCE}" (at 0.3 0) (layer "F.Fab")
-        (effects (font (size 1 1) (thickness 0.15)))
-    )
-    (pad "" thru_hole circle (at 0 0) (size 3.5 3.5) (drill 2.2) (layers "*.Cu" "*.Mask"))
-  )
   (footprint "swoop:M2_hole_4.2mm" (layer "F.Cu")
     (at 80.229546 112.73997)
@@
   (gr_line (start 63.279167 81.04401) (end 63.269824 127.424999)
     (stroke (width 0.05) (type solid)) (layer "Edge.Cuts"))
-  (gr_line (start 151.15 78.125) (end 151.15 72.125)
-    (stroke (width 0.05) (type solid)) (layer "Edge.Cuts"))
-  (gr_line (start 171.38563 81.989604) (end 171.385883 121.456747)
-    (stroke (width 0.05) (type solid)) (layer "Edge.Cuts"))
-  (gr_arc (start 169.385641 79.989462) (mid 170.799855 80.575345) (end 171.38563 81.989604)
+  (gr_line (start 151.154912 81.864669) (end 151.15 72.125)
+    (stroke (width 0.05) (type solid)) (layer "Edge.Cuts"))
+  (gr_line (start 171.374989 85.740125) (end 171.385883 121.456747)
+    (stroke (width 0.05) (type solid)) (layer "Edge.Cuts"))
+  (gr_arc (start 169.375 83.739983) (mid 170.789221 84.325861) (end 171.374989 85.740125)
     (stroke (width 0.05) (type solid)) (layer "Edge.Cuts"))
   (gr_line (start 131.95 67.825) (end 117.8 67.825)
@@
   (gr_arc (start 99.230865 63.020111) (mid 99.773567 61.783235) (end 101.025 61.275)
     (stroke (width 0.05) (type solid)) (layer "Edge.Cuts"))
-  (gr_arc (start 167.385329 83.239378) (mid 167.238879 83.592933) (end 166.885323 83.739379)
-    (stroke (width 0.05) (type solid)) (layer "Edge.Cuts"))
   (gr_line (start 115.235769 136.194832) (end 103.554156 136.29463)
     (stroke (width 0.05) (type solid)) (layer "Edge.Cuts"))
   (gr_line (start 78.875 79.288834) (end 65.083651 79.288834)
     (stroke (width 0.05) (type solid)) (layer "Edge.Cuts"))
-  (gr_line (start 167.385329 83.239378) (end 167.385505 81.989453)
-    (stroke (width 0.05) (type solid)) (layer "Edge.Cuts"))
   (gr_line (start 82.09686 129.229483) (end 65.025 129.229483)
     (stroke (width 0.05) (type solid)) (layer "Edge.Cuts"))
@@
   (gr_arc (start 114.309778 61.263163) (mid 115.546654 61.805865) (end 116.054889 63.057298)
     (stroke (width 0.05) (type solid)) (layer "Edge.Cuts"))
-  (gr_line (start 152.887029 80.012186) (end 154.604315 79.989915)
-    (stroke (width 0.05) (type solid)) (layer "Edge.Cuts"))
-  (gr_arc (start 154.604315 79.989915) (mid 156.018546 80.575773) (end 156.604299 81.990048)
-    (stroke (width 0.05) (type solid)) (layer "Edge.Cuts"))
   (gr_arc (start 149.404889 70.330865) (mid 150.641765 70.873567) (end 151.15 72.125)
     (stroke (width 0.05) (type solid)) (layer "Edge.Cuts"))
@@
   (gr_arc (start 115.235769 136.194832) (mid 132.832334 138.511576) (end 149.229607 145.303912)
     (stroke (width 0.05) (type solid)) (layer "Edge.Cuts"))
-  (gr_line (start 156.604299 81.990048) (end 156.60448 83.23998)
-    (stroke (width 0.05) (type solid)) (layer "Edge.Cuts"))
   (gr_arc (start 157.723414 149.341792) (mid 157.268009 149.691235) (end 156.698895 149.616311)
     (stroke (width 0.05) (type solid)) (layer "Edge.Cuts"))
-  (gr_arc (start 157.104479 83.739983) (mid 156.750923 83.593538) (end 156.60448 83.23998)
-    (stroke (width 0.05) (type solid)) (layer "Edge.Cuts"))
   (gr_arc (start 63.279167 81.04401) (mid 63.825 79.8) (end 65.083651 79.288834)
     (stroke (width 0.05) (type solid)) (layer "Edge.Cuts"))
-  (gr_arc (start 167.385505 81.989453) (mid 167.971363 80.575217) (end 169.385641 79.989462)
-    (stroke (width 0.05) (type solid)) (layer "Edge.Cuts"))
   (gr_arc (start 99.235484 65.499713) (mid 98.692782 66.736589) (end 97.441349 67.244824)
     (stroke (width 0.05) (type solid)) (layer "Edge.Cuts"))
@@
   (gr_line (start 97.441349 67.244824) (end 82.48217 67.244898)
     (stroke (width 0.05) (type solid)) (layer "Edge.Cuts"))
-  (gr_arc (start 152.887029 80.012186) (mid 151.620067 79.435338) (end 151.15 78.125)
+  (gr_arc (start 152.891941 83.751855) (mid 151.625 83.175) (end 151.154912 81.864669)
     (stroke (width 0.05) (type solid)) (layer "Edge.Cuts"))
   (gr_arc (start 65.025 129.229483) (mid 63.780991 128.68365) (end 63.269824 127.424999)
     (stroke (width 0.05) (type solid)) (layer "Edge.Cuts"))
-  (gr_line (start 157.104479 83.739983) (end 166.885323 83.739379)
+  (gr_line (start 152.891941 83.751855) (end 169.375 83.739983)
     (stroke (width 0.05) (type solid)) (layer "Edge.Cuts"))
   (gr_arc (start 82.09686 129.229483) (mid 93.37405 131.096101) (end 103.554156 136.29463)
