File: pcbs/3x5_2/arkenswoop/arkenswoop.kicad_pcb (KiCad board)
At the start: 2 copper layers, 113.1 x 89.8 mm, 52 parts, among them J1 TRRS, SW1 Choc, SW10 Choc, SW11 Choc, SW12 Choc, SW13 Choc, SW14 Choc, SW15 Choc, SW16 Choc, SW17 Choc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

Commit message: moved the standard Arkenswoop to pcbs/3x5_2
Other:
- board text added: "${TITLE} v${REVISION} ${COMMENT1}"
- board text removed: "Arkenswoop v0.6.0 https://github.com/SuperFola/arkenswoop"
Changed lines of the file:
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@@
   (title_block
     (title "Arkenswoop")
-    (date "2023-06-25")
+    (date "2023-07-09")
     (rev "0.6.0")
     (company "SuperFola")
+    (comment 1 "https://github.com/SuperFola/arkenswoop")
   )
   (layers
@@
     (fp_arc (start -7.1 2) (mid -6.924265 1.575736) (end -6.5 1.4)
       (stroke (width 0.15) (type solid)) (layer "B.SilkS"))
-    (fp_arc (start -6.530356 6.099232) (mid -6.934864 5.913392) (end -7.1 5.5)
+    (fp_arc (start -6.530356 6.099232) (mid -6.934863 5.913392) (end -7.1 5.5)
       (stroke (width 0.15) (type solid)) (layer "B.SilkS"))
     (fp_arc (start -3.5 1.4) (mid -2.863604 1.663604) (end -2.6 2.3)
@@
   (gr_arc (start 79.547715 67.826168) (mid 80.093555 66.582164) (end 81.352199 66.070992)
     (stroke (width 0.05) (type solid)) (layer "Edge.Cuts"))
-  (gr_text "Arkenswoop v0.6.0\nhttps://github.com/SuperFola/arkenswoop" (at 166.084013 89.964022 90) (layer "B.SilkS")
+  (gr_text "${TITLE} v${REVISION}\n${COMMENT1}" (at 166.084013 89.964022 90) (layer "B.SilkS")
     (effects (font (size 0.8 0.8) (thickness 0.1)) (justify left mirror))
   )
@@
     (effects (font (size 0.9 0.9) (thickness 0.1)) (justify left bottom))
   )
-  (gr_text "Arkenswoop v0.6.0\nhttps://github.com/SuperFola/arkenswoop" (at 166.084012 114.024024 90) (layer "F.SilkS")
+  (gr_text "${TITLE} v${REVISION}\n${COMMENT1}" (at 166.084012 114.024024 90) (layer "F.SilkS")
     (effects (font (size 0.8 0.8) (thickness 0.1)) (justify left))
   )

Commit message: redoing the switch plates cutouts and adding a proper kicad library
Parts:
- removed EN1: RotaryEncoder_Switch, swoop:RotaryEncoder
- removed the H4 at (134.2, 103.8)
- BT1: footprint swoop:Battery_pads_reversible -> arkenswoop:Battery_pads_reversible
- D1, D10, D11, D12, D13, D14, D15, D16, D17, D2, D3, D4, D5, D6, D7, D8, D9, ED1: footprint swoop:D3_SMD -> arkenswoop:D3_SMD
- EN2: footprint swoop:RollerEncoder -> arkenswoop:RollerEncoder
- G***: footprint Library:erebor_silk -> arkenswoop:erebor_silk
- H1, H2, H3, H4: footprint swoop:M2_hole_4.2mm -> arkenswoop:M2_hole_4.2mm
- J1: footprint swoop:TRRS-3pin -> arkenswoop:TRRS-3pin
- O1: footprint swoop:OLED_jumpers -> arkenswoop:OLED_jumpers
- PSW1: footprint swoop:Power -> arkenswoop:Power
- RSW1: footprint swoop:Reset -> arkenswoop:Reset
- Ref** (x2): footprint chocolad:M2_hole_3.5mm -> arkenswoop:M2_hole_3.5mm
- Ref**: footprint swoop:M2_hole_3.5mm -> arkenswoop:M2_hole_3.5mm
- SW1, SW10, SW11, SW12, SW13, SW14, SW15, SW16, SW17, SW2, SW3, SW4, SW5, SW6, SW7, SW8, SW9: footprint Library:Kailh-pg1350-socket-reversible -> arkenswoop:Kailh-pg1350-socket-reversible
- U1: footprint swoop:ProMicro_jumpers -> arkenswoop:ProMicro_jumpers
Connections:
- D10 pad 2: Net-(D10-A) -> (no net)
- D12 pad 2: Net-(D12-A) -> (no net)
- D13 pad 2: Net-(D13-A) -> (no net)
- D14 pad 2: Net-(D14-A) -> (no net)
- D15 pad 2: Net-(D15-A) -> (no net)
- D16 pad 2: Net-(D16-A) -> (no net)
- D17 pad 2: Net-(D17-A) -> (no net)
- D2 pad 2: Net-(D2-A) -> (no net)
- D3 pad 2: Net-(D3-A) -> (no net)
- D4 pad 2: Net-(D4-A) -> (no net)
- D5 pad 2: Net-(D5-A) -> (no net)
- D7 pad 2: Net-(D7-A) -> (no net)
- D8 pad 2: Net-(D8-A) -> (no net)
- D9 pad 2: Net-(D9-A) -> (no net)
Routing:
- net col2: track 149.8 -> 141.9 mm
- net eda: track 78.8 -> 73.3 mm
- net edb: track 77.9 -> 72.6 mm
- net GND: track 164.2 -> 160.6 mm
- net er0: track 33.7 -> 31.3 mm
- net row2: track 123.3 -> 121.2 mm
- net col0: track 139.7 -> 137.6 mm
- net col1: track 112.9 -> 110.8 mm
- net col3: track 104.1 -> 105.1 mm
